Commit message: New launch file, teleop changes

File: description/robot_core.xacro (robot description, xacro)
@@ -41,4 +41,7 @@
         </xacro:inertial_box>
 	</link>
+    <gazebo reference="chassis">
+        <material>Gazebo/White</material>
+    </gazebo>
     <!-- LEFT WHEEL LINK -->
     <joint name="left_wheel_joint" type="continuous" >
@@ -64,4 +67,7 @@
         </xacro:inertial_cylinder>
     </link>
+    <gazebo reference="left_wheel">
+        <material>Gazebo/Blue</material>
+    </gazebo>
    <!-- RIGHT WHEEL LINK -->
     <joint name="right_wheel_joint" type="continuous" >
@@ -85,5 +91,9 @@
        <xacro:inertial_cylinder mass="0.1" length ="0.04" radius="0.05" >
             <origin xyz ="0 0 0" rpy = "0 0 0"/>
-       </xacro:inertial_cylinder>   </link>
+       </xacro:inertial_cylinder>
+    </link>
+    <gazebo reference="right_wheel">
+        <material>Gazebo/Blue</material>
+    </gazebo>
     <!-- CASTER WHEEL LINK -->
     <joint name = "caster_wheel_joint" type="fixed">
@@ -104,6 +114,13 @@
             </geometry>
        </collision>
-       <xacro:inertial_sphere mass="0.1" radius="0.05" >
+       <xacro:inertial_sphere mass="0.5" radius="0.05" >
             <origin xyz ="0 0 0" rpy = "0 0 0"/>
-       </xacro:inertial_sphere>   </link>
+       </xacro:inertial_sphere>
+    </link>
+ros2 run teleop_twist_keyboard  teleop_twist_keyboard
+    <gazebo reference="caster_wheel">
+        <material>Gazebo/Black</material>
+        <mu1 value="0.001"/>
+        <mu2 value="0.001"/>
+    </gazebo>
 </robot>
