Commit message: Changes for ro2_control

File: description/robot.urdf.xacro (robot description, xacro)
@@ -2,4 +2,7 @@
 <robot xmlns:xacro="http://www.ros.org/wiki/xacro"  name="robot">
     <xacro:include filename="robot_core.xacro" />
-    <xacro:include filename="gazebo_control.xacro" />
+    <!-- xacro:include filename="gazebo_control.xacro" /> -->
+    <xacro:include filename="ros2_control.xacro" />
+    <xacro:include filename="lidar.xacro"/>
+    <xacro:include filename="camera.xacro"/>
 </robot>

File: description/robot_core.xacro (robot description, xacro)
@@ -10,4 +10,7 @@
     <material name="blue" >
 		<color rgba="0.2 0.2 1 1" />
+	</material>
+    <material name="red" >
+		<color rgba="1 0 0 1" />
 	</material>
     <material name="black" >
@@ -118,5 +121,4 @@
        </xacro:inertial_sphere>
     </link>
-ros2 run teleop_twist_keyboard  teleop_twist_keyboard
     <gazebo reference="caster_wheel">
         <material>Gazebo/Black</material>
