Commit message: Changes to robot_core.xacro for real robot.

File: description/camera.xacro (robot description, xacro)
@@ -4,5 +4,5 @@
         <parent link="chassis"/>
 		<child link="camera_link"/>
-		<origin xyz="0.305 0 0.08" rpy="0 0 0"/>
+		<origin xyz="0.255 0 0.08" rpy="0 0 0"/>
 	</joint>
     <link name="camera_link">

File: description/lidar.xacro (robot description, xacro)
@@ -4,5 +4,5 @@
         <parent link="chassis"/>
 		<child link="laser_frame"/>
-		<origin xyz="0.1 0 0.175" rpy="0 0 0"/>
+		<origin xyz="0.1 0 0.120" rpy="0 0 0"/>
 	</joint>
     <link name="laser_frame">

File: description/robot.urdf.xacro (robot description, xacro)
@@ -1,5 +1,5 @@
 <?xml version="1.0"?>
 <robot xmlns:xacro="http://www.ros.org/wiki/xacro"  name="robot">
-    <xacro:include filename="robot_core.xacro" />
+    <xacro:include filename="robot_core_real2.xacro" />
     <!-- xacro:include filename="gazebo_control.xacro" /> -->
     <xacro:include filename="ros2_control.xacro" />

File: description/robot_core_real.xacro (robot description, xacro)
@@ -1,5 +1,6 @@
 <?xml version="1.0"?>
 <robot xmlns:xacro="http://www.ros.org/wiki/xacro">
-    <xacro:include filename="inertial_macros.xacro"/>
+   <xacro:include filename="inertial_macros.xacro"/>
+<!-- This version for gazebo, using real robot dimensions -->
     <material name="white" >
         <color rgba="1 1 1 1" />
@@ -23,23 +24,23 @@
         <parent link="base_link"/>
         <child link="chassis"/>
-        <origin xyz="-0.1 0 0"/>
+        <origin xyz="-0.063 0 0.02"/>
     </joint>
     <!-- CHASSIS LINK -->
     <link name="chassis">
         <visual>
-            <origin xyz="0.15 0 0.075"/>
+            <origin xyz="0.125 0 0.05"/>
             <geometry>
-                <box size="0.3 0.3 0.15"/>
+                <box size="0.25 0.2 0.1"/>
             </geometry>
             <material name="white"/>
         </visual>
         <collision>
-            <origin xyz="0.15 0 0.075"/>
+            <origin xyz="0.125 0 0.05"/>
             <geometry>
-                <box size="0.3 0.3 0.15"/>
+                <box size="0.25 0.2 0.1"/>
             </geometry>
         </collision>
-        <xacro:inertial_box mass="0.5" x="0.3" y="0.3" z="0.15" >
-            <origin xyz ="0.15 0 0.75" rpy = "0 0 0"/>
+        <xacro:inertial_box mass="0.5" x="0.25" y="0.2" z="0.1" >
+            <origin xyz ="0.125 0 0.05" rpy = "0 0 0"/>
         </xacro:inertial_box>
     </link>
@@ -51,5 +52,5 @@
         <parent link="base_link"/>
         <child link = "left_wheel"/>
-        <origin xyz="0 0.175 0" rpy="-${pi/2} 0 0"/>
+        <origin xyz="0 0.12 0" rpy="-${pi/2} 0 0"/>
         <axis xyz = "0 0 1" />
     </joint>
@@ -57,5 +58,5 @@
         <visual>
             <geometry>
-                <cylinder radius="0.05" length="0.04"/>
+                <cylinder radius="0.033" length="0.026"/>
             </geometry>
             <material name="blue"/>
@@ -63,8 +64,8 @@
         <collision>
             <geometry>
-                <cylinder radius="0.05" length="0.04"/>
+                <cylinder radius="0.033" length="0.026"/>
             </geometry>
         </collision>
-        <xacro:inertial_cylinder mass="0.1" length ="0.04" radius="0.05" >
+        <xacro:inertial_cylinder mass="0.1" length ="0.026" radius="0.033">
             <origin xyz ="0 0 0" rpy = "0 0 0"/>
         </xacro:inertial_cylinder>
@@ -73,9 +74,9 @@
         <material>Gazebo/Blue</material>
     </gazebo>
-   <!-- RIGHT WHEEL LINK -->
+    <!-- RIGHT WHEEL LINK -->
     <joint name="right_wheel_joint" type="continuous" >
         <parent link="base_link"/>
         <child link = "right_wheel"/>
-        <origin xyz="0 -0.175 0" rpy="${pi/2} 0 0"/>
+        <origin xyz="0 -0.12 0" rpy="${pi/2} 0 0"/>
         <axis xyz = "0 0 -1" />
     </joint>
@@ -83,5 +84,5 @@
         <visual>
             <geometry>
-                <cylinder radius="0.05" length="0.04"/>
+                <cylinder radius="0.033" length="0.026"/>
             </geometry>
             <material name="blue"/>
@@ -89,8 +90,8 @@
         <collision>
             <geometry>
-                <cylinder radius="0.05" length="0.04"/>
+                <cylinder radius="0.033" length="0.026"/>
             </geometry>
        </collision>
-       <xacro:inertial_cylinder mass="0.1" length ="0.04" radius="0.05" >
+       <xacro:inertial_cylinder mass="0.1" length ="0.026" radius="0.033" >
             <origin xyz ="0 0 0" rpy = "0 0 0"/>
        </xacro:inertial_cylinder>
@@ -103,10 +104,10 @@
         <parent link="chassis"/>
         <child link="caster_wheel"/>
-        <origin xyz="0.24 0 0"/>
+        <origin xyz="0.2 0 -0.02"/>
     </joint>
     <link name = "caster_wheel">
         <visual>
             <geometry>
-                <sphere radius="0.05" />
+                <sphere radius="0.033" />
             </geometry>
             <material name="black"/>
@@ -114,8 +115,8 @@
        <collision>
             <geometry>
-                <sphere radius="0.05" />
+                <sphere radius="0.033" />
             </geometry>
        </collision>
-       <xacro:inertial_sphere mass="0.5" radius="0.05" >
+       <xacro:inertial_sphere mass="0.5" radius="0.033" >
             <origin xyz ="0 0 0" rpy = "0 0 0"/>
        </xacro:inertial_sphere>
