Commit message: Changes for 130 RPM motor

File: description/robot_core_real2.xacro (robot description, xacro)
@@ -12,8 +12,8 @@
     <xacro:property name="wheel_offset_y" value="0.120"/>
     <xacro:property name="wheel_offset_z" value="0.02"/>
-    <xacro:property name="caster_wheel_radius" value="0.033"/>
+    <xacro:property name="caster_wheel_radius" value="0.01"/>
     <xacro:property name="caster_wheel_mass" value="0.01"/>
-    <xacro:property name="caster_wheel_offset_x" value="0.2"/>
-    <xacro:property name="caster_wheel_offset_z" value="-0.020"/>
+    <xacro:property name="caster_wheel_offset_x" value="0.170"/>
+    <xacro:property name="caster_wheel_offset_z" value="-0.040"/>
     <material name="white">
         <color rgba="1 1 1 1" />
@@ -46,5 +46,5 @@
         <parent link="base_link"/>
         <child link="chassis"/>
-        <origin xyz="${-wheel_offset_x} 0 ${wheel_offset_z}"/>
+        <origin xyz="${-wheel_offset_x} 0 ${-wheel_offset_z}"/>
     </joint>
     <link name="chassis">

File: description/ros2_control.xacro (robot description, xacro)
@@ -11,5 +11,5 @@
                 <param name="baud_rate">57600</param>
                 <param name="timeout_ms">1000</param>
-                <param name="enc_counts_per_rev">660</param>
+                <param name="enc_counts_per_rev">1906</param>
             </hardware>
             <joint name="left_wheel_joint">

Commit message: Final changes, Nav2 etc

File: description/robot_core_real2.xacro (robot description, xacro)
@@ -11,5 +11,5 @@
     <xacro:property name="wheel_offset_x" value="0.063"/>
     <xacro:property name="wheel_offset_y" value="0.120"/>
-    <xacro:property name="wheel_offset_z" value="0.02"/>
+    <xacro:property name="wheel_offset_z" value="-0.02"/>
     <xacro:property name="caster_wheel_radius" value="0.01"/>
     <xacro:property name="caster_wheel_mass" value="0.01"/>
